Commit message: Pioneer with camera

File: p2os_urdf/defs/pioneer3at.xacro (robot description, xacro)
@@ -11,3 +11,63 @@
 <xacro:p3at_back suffix="right" reflect="-1"/>
 <xacro:p3at_gazebo_ext/>
+	<xacro:property name="cameraSize" value="0.05"/>
+	<xacro:property name="cameraMass" value="0.1"/>
+	<joint name="fixed_camera" type="fixed">
+	  <parent link="base_link"/>
+	  <child link="cam"/>
+          <origin rpy="0 0 0" xyz="0.25 0 0.3"/>
+	</joint>
+	<link name="cam">
+	  <collision>
+	    <origin xyz="0 0 0" rpy="0 0 0"/>
+	    <geometry>
+	      <box size="${cameraSize} ${cameraSize} ${cameraSize}"/>
+	    </geometry>
+	  </collision>
+	  <visual>
+	    <origin xyz="0 0 0" rpy="0 0 0"/>
+	    <geometry>
+	      <box size="${cameraSize} ${cameraSize} ${cameraSize}"/>
+	    </geometry>
+	    <material name="blue"/>
+	  </visual>
+	  <inertial>
+	    <mass value="${cameraMass}" />
+	    <origin xyz="0 0 0" rpy="0 0 0"/>
+			<inertia ixx="0.012411765597" ixy="0" ixz="0"
+         iyy="0.015218160428" iyz="0" izz="0.011763977943"/>
+	  </inertial>
+	</link>
+	<gazebo reference="cam">
+	  <material>Gazebo/Blue</material>
+	  <sensor type="camera" name="cam">
+	    <update_rate>30.0</update_rate>
+	    <camera name="head">
+	      <horizontal_fov>1.3962634</horizontal_fov>
+	      <image>
+		<width>800</width>
+		<height>800</height>
+		<format>R8G8B8</format>
+	      </image>
+	      <clip>
+		<near>0.02</near>
+		<far>300</far>
+	      </clip>
+	    </camera>
+	    <plugin name="camera_controller" filename="libgazebo_ros_camera.so">
+	      <alwaysOn>true</alwaysOn>
+	      <updateRate>0.0</updateRate>
+	      <cameraName>pioneer3at/camera1</cameraName>
+	      <imageTopicName>image_raw</imageTopicName>
+	      <cameraInfoTopicName>camera_info</cameraInfoTopicName>
+	      <frameName>camera_link</frameName>
+	      <hackBaseline>0.07</hackBaseline>
+	      <distortionK1>0.0</distortionK1>
+	      <distortionK2>0.0</distortionK2>
+	      <distortionK3>0.0</distortionK3>
+	      <distortionT1>0.0</distortionT1>
+	      <distortionT2>0.0</distortionT2>
+	    </plugin>
+	  </sensor>
+	 </gazebo>
 </robot>

Commit message: IR sensor integrated.

File: p2os_urdf/defs/pioneer3at.xacro (robot description, xacro)
@@ -72,3 +72,65 @@
 	  </sensor>
 	 </gazebo>
+	<joint name="ir_front_joint" type="fixed">
+    <axis xyz="0 1 0" />
+    <origin rpy="0 0 0" xyz="0.25 0 0.4" />
+    <parent link="base_link"/>
+    <child link="base_ir_front"/>
+	</joint>
+	<link name="base_ir_front">
+	    <collision>
+	      <origin xyz="0 0 0" rpy="0 0 0"/>
+	      <geometry>
+	        <box size="0.01 0.01 0.01"/>
+	      </geometry>
+	    </collision>
+	    <visual>
+	      <origin xyz="0 0 0" rpy="0 0 0"/>
+	      <geometry>
+	        <box size="0.1 0.1 0.1"/>
+	      </geometry>
+	    </visual>
+	    <inertial>
+	      <mass value="1e-5" />
+	      <origin xyz="0 0 0" rpy="0 0 0"/>
+	      <inertia ixx="1e-6" ixy="0" ixz="0" iyy="1e-6" iyz="0"      izz="1e-6" />
+	    </inertial>
+	</link>
+	<gazebo reference="base_ir_front">
+   <sensor type="ray" name="TeraRanger">
+      <pose>0 0 0 0 0 0</pose>
+      <visualize>true</visualize>
+      <update_rate>50</update_rate>
+      <ray>
+         <scan>
+            <horizontal>
+               <samples>10</samples>
+               <resolution>1</resolution>
+               <min_angle>-0.14835</min_angle>
+               <max_angle>0.14835</max_angle>
+            </horizontal>
+            <vertical>
+               <samples>10</samples>
+               <resolution>1</resolution>
+               <min_angle>-0.14835</min_angle>
+               <max_angle>0.14835</max_angle>
+            </vertical>
+         </scan>
+         <range>
+            <min>0.01</min>
+            <max>2</max>
+            <resolution>0.02</resolution>
+         </range>
+      </ray>
+      <plugin filename="libgazebo_ros_range.so" name="gazebo_ros_range">
+         <gaussianNoise>0.005</gaussianNoise>
+         <alwaysOn>true</alwaysOn>
+         <updateRate>50</updateRate>
+         <topicName>sensor/ir_front</topicName>
+         <frameName>base_ir_front</frameName>
+         <radiation>INFRARED</radiation>
+         <fov>0.2967</fov>
+      </plugin>
+   </sensor>
+   </gazebo>
 </robot>

Commit message: Create map working.

File: p2os_urdf/defs/pioneer3at.xacro (robot description, xacro)
@@ -74,5 +74,5 @@
 	<joint name="ir_front_joint" type="fixed">
     <axis xyz="0 1 0" />
-    <origin rpy="0 0 0" xyz="0.25 0 0.4" />
+    <origin rpy="0 0 0" xyz="0 0 0.4" />
     <parent link="base_link"/>
     <child link="base_ir_front"/>
